Commit message: loaf

File: src/control_pkg/ros2_control_config/control.ros2_control.xacro (robot description, xacro)
@@ -4,5 +4,5 @@
         <hardware>
             <plugin>mujoco_ros2_control/MujocoSystemInterface</plugin>
-            <param name="mujoco_model">$(find descrip_pkg)/urdf/White_Tigger.xml</param>
+            <param name="mujoco_model">$(find descrip_pkg)/urdf/go2.xml</param>
             <param name="sim_speed_factor">1.0</param>
             <param name="initial_keyframe">init_pose</param>

File: src/descrip_pkg/urdf/small_dog_copy.urdf (robot description, URDF)
Before this commit: robot small_dog, 17 links, 16 joints
Links:
- link base_link: geometry collision mesh filename=meshes/base_link.stl; visual mesh filename=meshes/base_link.stl
- link bl_calf_Link: geometry collision mesh filename=meshes/bl_calf_Link.stl; visual mesh filename=meshes/bl_calf_Link.stl
- link bl_foot_Link: geometry collision mesh filename=meshes/bl_foot_Link.stl; visual mesh filename=meshes/bl_foot_Link.stl
- link bl_hip_Link: geometry collision mesh filename=meshes/bl_hip_Link.stl; visual mesh filename=meshes/bl_hip_Link.stl
- link bl_thigh_Link: geometry collision mesh filename=meshes/bl_thigh_Link.stl; visual mesh filename=meshes/bl_thigh_Link.stl
- link br_calf_Link: geometry collision mesh filename=meshes/br_calf_Link.stl; visual mesh filename=meshes/br_calf_Link.stl
- link br_foot_Link: geometry collision mesh filename=meshes/br_foot_Link.stl; visual mesh filename=meshes/br_foot_Link.stl
- link br_hip_Link: geometry collision mesh filename=meshes/br_hip_Link.stl; visual mesh filename=meshes/br_hip_Link.stl
- link br_thigh_Link: geometry collision mesh filename=meshes/br_thigh_Link.stl; visual mesh filename=meshes/br_thigh_Link.stl
- link fl_calf_Link: geometry collision mesh filename=meshes/fl_calf_Link.stl; visual mesh filename=meshes/fl_calf_Link.stl
- link fl_foot_Link: geometry collision mesh filename=meshes/fl_foot_Link.stl; visual mesh filename=meshes/fl_foot_Link.stl
- link fl_hip_Link: geometry collision mesh filename=meshes/fl_hip_Link.stl; visual mesh filename=meshes/fl_hip_Link.stl
- link fl_thigh_Link: geometry collision mesh filename=meshes/fl_thigh_Link.stl; visual mesh filename=meshes/fl_thigh_Link.stl
- link fr_calf_Link: geometry collision mesh filename=meshes/fr_calf_Link.stl; visual mesh filename=meshes/fr_calf_Link.stl
- link fr_foot_Link: geometry collision mesh filename=meshes/fr_foot_Link.stl; visual mesh filename=meshes/fr_foot_Link.stl
- link fr_hip_Link: geometry collision mesh filename=meshes/fr_hip_Link.stl; visual mesh filename=meshes/fr_hip_Link.stl
- link fr_thigh_Link: geometry collision mesh filename=meshes/fr_thigh_Link.stl; visual mesh filename=meshes/fr_thigh_Link.stl
Joints:
- joint bl_hip_joint: axis -1 0 0 -> 1 0 0
- joint br_hip_joint: axis -1 0 0 -> 1 0 0
- joint fl_hip_joint: axis -1 0 0 -> 1 0 0
- joint fr_hip_joint: axis -1 0 0 -> 1 0 0

File: src/descrip_pkg/urdf/total.urdf.xacro (robot description, xacro)
@@ -1,5 +1,5 @@
 <?xml version="1.0"?>
 <robot xmlns:xacro="http://www.ros.org/wiki/xacro" name="White_Tigger">
-  <xacro:include filename="$(find descrip_pkg)/urdf/small_dog.urdf"/>
+  <xacro:include filename="$(find descrip_pkg)/urdf/go2_description.urdf"/>
   <xacro:include filename="$(find control_pkg)/ros2_control_config/control.ros2_control.xacro"/>
 </robot>
